Commit message: robot localization with gps, imu and wheel odometry

File: ugv_gazebo_sim/hunter_se/hunter_se_description/urdf/hunter_se_description.urdf (robot description, URDF)
Before this commit: robot hunter_se_description, 14 links, 13 joints
Links:
- added link imu_link, mass 1e-5; collision box size=0.2 0.2 0.05; visual box size=0.2 0.2 0.05
Joints:
- added joint imu_joint: type fixed, parent base_link, child imu_link, origin xyz=-0.10 0 0 rpy=-0 0 0
